File: Kicad Project/YX55069BCT2-Driver-Board.kicad_sch (KiCad schematic)
At the start: 0 parts

Commit message: wired up esp32 + almost done with HDMI -> MIPI Converter
Parts:
- added C1, C17, C19, C20, C22, C23, C25, C26, C28, C3: 4.7 µF, YX55069BCT2:C_0603_1608Metric, symbol Device:C_Small
- added C10: 1.0µF, Capacitor_SMD:C_0603_1608Metric, symbol Device:C_Small
- added C11: 10µF, Capacitor_SMD:C_0603_1608Metric, symbol Device:C_Small
- added C12: 2.2µF, Capacitor_SMD:C_0603_1608Metric, symbol Device:C_Small
- added C13: 4.7µF, Capacitor_SMD:C_0603_1608Metric, symbol Device:C_Small
- added C14, C15, C36, C4, C5, C7, C8, C9: 100nF, YX55069BCT2:C0603, symbol Device:C_Small
- added C147: 100nF, Capacitor_SMD:C_0603_1608Metric, symbol Device:C_Small
- added C150, C155: 1µF, Capacitor_SMD:C_0603_1608Metric, symbol Device:C_Small
- added C156: 100pF, Capacitor_SMD:C_0603_1608Metric, symbol Device:C_Small
- added C18, C2, C21, C24, C27: 100 nF, YX55069BCT2:C_0603_1608Metric, symbol Device:C_Small
- added C31, C33, C34, C35: 10uF, YX55069BCT2:C0603, symbol Device:C_Small
- added C32: 1uF, YX55069BCT2:CL05A105KA5NQNC, symbol Device:C_Small
- added C37, C38: 15 pF, YX55069BCT2:C0402, symbol Device:C_Small
- added C6: 100nf, YX55069BCT2:C0603, symbol Device:C_Small
- added D2: S16, YX55069BCT2:SOD-123FL_L2.7-W1.8-LS3.8-RD, symbol YX55069BCT2:S16
- added FB1, FB2: FerriteBead, YX55069BCT2:USB-C-SMD_TYPE-C16PIN, symbol Device:FerriteBead
- added FPC1: FPC0.5-24P, slate113:FPC-SMD_P0.50-24P_XJ-FGS, symbol slate113:FPC0.5-24P
- added FPC2: FPC-0.5FX-6PWBH10, slate113:FPC-SMD_FPC-0.5FX-6PWBH10, symbol slate113:FPC-0.5FX-6PWBH10
- added J1: 10029449-001RLF, YX55069BCT2:HDMI_A_Amphenol_10029449-x01xLF_Horizontal, symbol YX55069BCT2:10029449-001RLF
- added J2: Conn_01x06_Pin, Package_DFN_QFN:QFN-20-1EP_5x5mm_P0.65mm_EP3.35x3.35mm, symbol Connector:Conn_01x06_Pin
- added L3: 10µH, slate113:IND-SMD_L7.1-W6.6, symbol Device:L
- added OSC1: OT7EL89CJI-111YLC-48M, YX55069BCT2:OSC-SMD_4P-L2.0-W1.6-BL, symbol YX55069BCT2:OT7EL89CJI-111YLC-48M
- added Q1: BSS138_C112239, YX55069BCT2:SOT-23-3_L2.9-W1.6-P1.90-LS2.8-BR, symbol YX55069BCT2:BSS138_C112239
- added R1: 2.00 kOhm, YX55069BCT2:R0402, symbol YX55069BCT2:RC0402FR-072KL
- added R10: 127kΩ, Resistor_SMD:R_0603_1608Metric, symbol Device:R
- added R100, R102: 10kΩ, Resistor_SMD:R_0603_1608Metric, symbol Device:R
- added R101, R97, R98: 4.7kΩ, Resistor_SMD:R_0603_1608Metric, symbol Device:R
- added R105: 100kΩ, Resistor_SMD:R_0603_1608Metric, symbol Device:R_Small
- added R11, R2, R6, R7: 10 kOhm, YX55069BCT2:R0402, symbol YX55069BCT2:RC0402FR-0710KL
- added R12: 0 Ohm, YX55069BCT2:R0402, symbol YX55069BCT2:RC0402FR-070RL
- added R13: 22 Ohm, YX55069BCT2:R0402, symbol YX55069BCT2:RC0402FR-0722RL
- added R22: 100 Ohm, YX55069BCT2:R0402, symbol YX55069BCT2:RC0402FR-07100RL
- added R3: 49.9 kΩ, Resistor_THT:R_Array_SIP4, symbol Device:R_Small
- added R4, R5: 100 kΩ, Resistor_THT:R_Array_SIP4, symbol Device:R_Small
- added R8: 205kΩ, Resistor_SMD:R_0603_1608Metric, symbol Device:R
- added R9: 37.4 kΩ, Resistor_THT:R_Array_SIP4, symbol Device:R_Small
- added R96: 10kΩ, Resistor_SMD:R_0603_1608Metric, symbol Device:R_Small
- added R99: 200kΩ, Resistor_SMD:R_0603_1608Metric, symbol Device:R_Small
- added SW3: BOOT, slate113:KEY-SMD_KMR2XXGXXX, symbol Switch:SW_Push
- added SW4: RESET, slate113:KEY-SMD_KMR2XXGXXX, symbol Switch:SW_Push
- added U1: TC358870XBG(NOK), YX55069BCT2:P-VFBGA-80_L7.0-W7.0-R10-C10-P0.65-TL, symbol YX55069BCT2:TC358870XBG(NOK)
- added U10: ESP32-S3R8, YX55069BCT2:QFN-56_L7.0-W7.0-P0.40-TL-EP4.0, symbol YX55069BCT2:ESP32-S3R8
- added U11: GD25Q128EWIGR, YX55069BCT2:WSON-8_L6.0-W5.0-P1.27-TL-EP, symbol YX55069BCT2:GD25Q128EWIGR
- added U12: USBLC6-2SC6, Package_TO_SOT_SMD:SOT-23-6, symbol Power_Protection:USBLC6-2SC6
- added U2, U7: TLV76701DRVR, YX55069BCT2:WSON-6_L2.0-W2.0-P0.65-TL-EP, symbol YX55069BCT2:TLV76701DRVR
- added U3: CH224K, Package_SO:SSOP-10-1EP_3.9x4.9mm_P1mm_EP2.1x3.3mm, symbol Interface_USB:CH224K
- added U4: TLV76718DRVR, YX55069BCT2:WSON-6_L2.0-W2.0-P0.65-BL-EP, symbol YX55069BCT2:TLV76718DRVR
- added U5: TLV76728DRVR, YX55069BCT2:WSON-6_L2.0-W2.0-P0.65-BL-EP, symbol YX55069BCT2:TLV76728DRVR
- added U6: TLV76733DRVR, YX55069BCT2:WSON-6_L2.0-W2.0-P0.65-TL-EP, symbol YX55069BCT2:TLV76733DRVR
- added U62: PCA9306DCUR, slate113:SSOP-8_L2.0-W2.3-P0.50-LS3.1-BR, symbol slate113:PCA9306DCUR
- added U63: AP2120N-2.8TRG1, slate113:SOT-23-3_L2.9-W1.3-P1.90-LS2.4-BR, symbol slate113:AP2120N-2.8TRG1
- added U8: ESD7104MUTAG_C2987068, slate113:DFN-10_L2.5-W1.0-P0.50-BL, symbol slate113:ESD7104MUTAG_C2987068
- added U9: LP8556SQ-E09/NOPB, slate113:WQFN-24_L4.0-W4.0-P0.50-BL-EP2.5, symbol slate113:LP8556SQ-E09_NOPB
- added USB1: TYPE-C16PIN, YX55069BCT2:USB-C-SMD_TYPE-C16PIN, symbol YX55069BCT2:TYPE-C16PIN
- added X1: ABM8-40.000MHZ-10-D1G-T, YX55069BCT2:CRYSTAL-SMD_4P-L3.2-W2.5-BL, symbol YX55069BCT2:ABM8-40.000MHZ-10-D1G-T
Connections:
- new net: FB1.1, J1.SH
- new net: C21.1, U6.2 (FB)
- new net: C18.1, R3.1, R4.2, U2.2 (FB)
- new net: OSC1.1 (Tri-state), R2.2
- new net: C8.2, U1.J1 (BIASDA)
- new net: C24.1, U4.2 (FB)
- new net: OSC1.3 (OUT), R13.1
- new net: C27.1, R5.2, R9.1, U7.2 (FB)
- new net: FB2.1, USB1.1 (SHELL), USB1.2 (SHELL), USB1.3 (SHELL), USB1.4 (SHELL)
- new net: R10.1, U9.23 (ISET)
- new net: C38.2, R12.2, X1.1 (OSC1)
- new net: C37.2, U10.53 (XTAL_N), X1.3 (OSC2)
- new net: R1.1, U1.A1 (REXT)
- new net: R13.2, U1.K9 (REFCLK)
- new net: Q1.1 (G), R105.2, R22.1
- new net: C14.2, U1.K2 (PFIL)
- new net: C156.1, R99.1, U62.7 (VREF2), U62.8 (EN)
- new net: C9.2, U1.K1 (PCKIN)
- new net: Q1.3 (D), R11.1, U1.K8 (RESETN)
- new net: R12.1, U10.54 (XTAL_P)
- new net: C2.1, U5.2 (FB)
- new net: R8.1, U9.21 (FSET)
- new net: C11.1, U9.19 (VLDO)
- new net 1V1: C26.2, C27.2, R9.2, U7.1 (OUT)
- new net 1V2: C17.2, C18.2, R3.2, U2.1 (OUT)
- new net 1V8: C15.2, C23.2, C24.2, FPC1.22, OSC1.4 (VDD), R100.2, R11.2, R2.1, R96.1, R97.2, R98.1, U4.1 (OUT), U62.2 (VREF1)
- new net 2V8: C2.2, C3.2, U5.1 (OUT)
- new net CC1: U3.7 (CC1), USB1.A5 (CC1)
- new net CC2: U3.6 (CC2), USB1.B5 (CC2)
- new net CHIP_PU: C32.2, R6.2, SW4.1, U10.4 (CHIP_PU)
- new net D0+: J1.7 (D0+), U1.D1 (HDMID0P)
- new net D0-: J1.9 (D0-), U1.D2 (HDMID0N)
- new net D1+: J1.4 (D1+), U1.E1 (HDMID1P)
- new net D1-: J1.6 (D1-), U1.E2 (HDMID1N)
- new net D2+: J1.1 (D2+), U1.F1 (HDMID2P)
- new net D2-: J1.3 (D2-), U1.F2 (HDMID2N)
- new net DDC_SCL: J1.15 (SCL), U1.A3 (DDC_SCL)
- new net DDC_SDA: J1.16 (SDA), U1.B3 (DDC_SDA)
- new net DSI_CLKN: FPC1.9, U1.F9 (CDSI0CN)
- new net DSI_CLKP: FPC1.10, U1.F10 (CDSI0CP)
- new net DSI_D0N: FPC1.6, U1.H9 (CDSI0D0N)
- new net DSI_D0P: FPC1.7, U1.H10 (CDSI0D0P)
- new net DSI_D1N: FPC1.12, U1.G9 (CDSI0D1N)
- new net DSI_D1P: FPC1.13, U1.G10 (CDSI0D1P)
- new net DSI_D2N: FPC1.15, U1.E9 (CDSI0D2N)
- new net DSI_D2P: FPC1.16, U1.E10 (CDSI0D2P)
- new net DSI_D3N: FPC1.3, U1.D9 (CDSI0D3N)
- new net DSI_D3P: FPC1.4, U1.D10 (CDSI0D3P)
- new net ESP_DN: U10.25 (GPIO19), U12.4 (I/O2)
- new net ESP_DP: U10.26 (GPIO20), U12.6 (I/O1)
- new net GND: C1.2, C10.1, C10.2, C11.2, C12.1, C12.2, C13.2, C14.1, C147.2, C15.1, C150.1, C150.2, C155.1, C156.2, C17.1, C19.2, C20.1, C20.2, C21.2, C22.2, C23.1, C25.2, C26.1, C28.2, C3.1, C31.1, C31.2, C32.1, C33.1, C33.2, C34.1, C34.2, C35.1, C35.2, C36.1, C36.2, C37.1, C38.1, C4.1, C4.2, C5.1, C5.2, C6.1, C6.2, C7.1, C8.1, C9.1, FB1.2, FB2.2, FPC1.11, FPC1.14, FPC1.17, FPC1.2, FPC1.23, FPC1.24, FPC1.25, FPC1.26, FPC1.5, FPC1.8, FPC2.6, FPC2.7, FPC2.8, J1.11 (CKS), J1.17 (GND), J1.2 (D2S), J1.5 (D1S), J1.8 (D0S), L3.1, OSC1.2 (GND), Q1.2 (S), R10.2, R101.2, R102.2, R105.1, R4.1, R5.1, R6.1, R7.1, R8.2, R99.2, SW3.2, SW4.2, U1.G5 (TEST), U1.G6 (IR), U10.2 (VDD3P3), U10.20 (VDD3P3_RTC), U10.3 (VDD3P3), U10.46 (VDD3P3_CPU), U10.55 (VDDA), U10.56 (VDDA), U10.57 (GND), U11.4 (VSS), U11.9 (EP), U12.2 (GND), U2.3 (GND), U2.5 (GND), U2.7 (EP), U3.1 (VDD), U3.11 (GND), U3.2 (CFG2), U3.3 (CFG3), U3.9 (CFG1), U4.3 (GND), U4.5 (GND), U4.7 (EP), U5.3 (GND), U5.5 (GND), U5.7 (EP), U6.1 (OUT), U6.3 (GND), U6.5 (GND), U6.7 (EP), U62.1 (GND), U63.1 (GND), U63.3 (VIN), U7.3 (GND), U7.5 (GND), U7.7 (EP), U8.3, U8.8, U9.10 (GND), U9.11 (GND), U9.15 (GND), U9.22 (VDD), U9.24 (GND), U9.25 (EP), U9.3 (GND_SW), U9.4 (GND_SW), U9.7 (EN/VDDIO), USB1.A1B12 (GND), USB1.B1A12 (GND), X1.2 (GND), X1.4 (GND)
- new net GPIO0: R7.2, SW3.1, U10.5 (GPIO0)
- new net HDMICN: J1.12 (CK-), U1.C2 (HDMICN)
- new net HDMICP: J1.10 (CK+), U1.C1 (HDMICP)
- new net HDMI_5V_IN: J1.18 (+5V), U1.A4 (HPDI)
- new net HPD0: J1.19 (HPD), U1.B4 (HPDO)
- new net I2C0_SCL: R102.1, U1.K4 (I2C_SCL), U10.10 (GPIO5), U62.6 (SCL2), U9.6 (SCL)
- new net I2C0_SDA: R101.1, U1.K3 (I2C_SDA), U10.9 (GPIO4), U62.5 (SDA2), U9.5 (SDA)
- new net L1P1: D2.2 (A), L3.2, U9.1 (SW), U9.2 (SW)
- new net LCD_LED_A: C13.1, D2.1 (C), FPC1.21, U9.20 (VBOOST)
- new net LCD_LED_K: FPC1.20, U9.12 (LED1), U9.13 (LED2)
- new net LCD_PWM: FPC1.18, U9.9 (PWM)
- new net LCD_RST_L: C147.1, FPC1.19, R96.2
- new net RESETN: R22.2, U10.11 (GPIO6)
- new net SPICLK: U10.33 (SPICLK), U11.6 (SCLK)
- new net SPICS0: U10.32 (SPICS0), U11.1 (~{CS})
- new net SPIDI: U10.35 (SPID), U11.5 (SI(IO0))
- new net SPIHOLD: U10.30 (SPIHD), U11.7 (~{HOLD}/RESET#(IO3))
- new net SPIQ: U10.34 (SPIQ), U11.2 (SO(IO1))
- new net SPIWP: U10.31 (SPIWP), U11.3 (WP#(IO2))
- new net TP_2V8: C155.2, FPC2.1, U63.2 (VOUT)
- new net TP_INT_L: FPC2.5, U10.7 (GPIO2), U8.5
- new net TP_RST_L: FPC2.3, R100.1, U10.6 (GPIO1), U8.2
- new net TP_SCL_1V8: FPC2.2, R98.2, U62.3 (SCL1), U8.1
- new net TP_SDA_1V8: FPC2.4, R97.1, U62.4 (SDA1), U8.4
- new net USB_DN: U12.1 (I/O1), USB1.A7 (DN1), USB1.B7 (DN2)
- new net USB_DP: U12.3 (I/O2), USB1.A6 (DP1), USB1.B6 (DP2)
- new net VBUS: C1.1, C19.1, C22.1, C25.1, C28.1, U12.5 (VBUS), U2.4 (EN), U2.6 (IN), U3.8 (VBUS), U4.4 (EN), U4.6 (IN), U5.4 (EN), U5.6 (IN), U6.4 (EN), U6.6 (IN), U7.4 (EN), U7.6 (IN), USB1.A4B9 (VBUS), USB1.B4A9 (VBUS)
- new net VDD33_HDMI: R1.2, U1.B1 (VDD33_HDMI)
- new net VDD_SPI: C7.2, U10.29 (VDD_SPI), U11.8 (VCC)
- no-connect marks 0 -> 25
Other:
- note added: "2V8 LDO"
- note added: "Backlight LED Driver"
- note added: "Display Clamshell"
- note added: "HDMI"
- note added: "I2C Pullups"
- note added: "LDOs"
- note added: "Level Shifter"
- note added: "Misc"
- note added: "Reset + Boot Buttons"
- note added: "SPI"
- note added: "TVS"
- note added: "Touch Clamshell"
- note added: "USB-C Diode"

Commit message: wired up remaining components
Parts:
- removed J2: Conn_01x06_Pin, Package_DFN_QFN:QFN-20-1EP_5x5mm_P0.65mm_EP3.35x3.35mm, symbol Connector:Conn_01x06_Pin
- removed R102: 10kΩ, Resistor_SMD:R_0603_1608Metric, symbol Device:R
- removed R9: 37.4 kΩ, Resistor_THT:R_Array_SIP4, symbol Device:R_Small
- added C157: 100pF, Capacitor_SMD:C_0603_1608Metric, symbol Device:C_Small
- added C16, C29, C30, C39, C40, C41, C42, C43, C44, C45, C46, C47, C59, C62: 100nF, YX55069BCT2:C0603, symbol Device:C_Small
- added C48, C58: 10uF, YX55069BCT2:C0603, symbol Device:C_Small
- added C49, C50, C51, C52, C61: 1uF, YX55069BCT2:C0603, symbol Device:C_Small
- added C53, C54, C55, C56, C57, C60: 2.2uF, YX55069BCT2:C0603, symbol Device:C_Small
- added D3: TPD4E05U06DQAR, YX55069BCT2:USON-10_L2.5-W1.0-P0.50-BL, symbol YX55069BCT2:TPD4E05U06DQAR
- added D4, D5: TPD4E02B04DQAR, YX55069BCT2:USON-10_L2.5-W1.0-P0.50-BL, symbol YX55069BCT2:TPD4E02B04DQAR
- added Q2: BSS138_C112239, YX55069BCT2:SOT-23-3_L2.9-W1.6-P1.90-LS2.8-BR, symbol YX55069BCT2:BSS138_C112239
- added R103: 200kΩ, Resistor_SMD:R_0603_1608Metric, symbol Device:R_Small
- added R104, R106, R108: 4.7kΩ, Resistor_SMD:R_0603_1608Metric, symbol Device:R
- added R107: 100kΩ, Resistor_SMD:R_0603_1608Metric, symbol Device:R_Small
- added R14: 10 kOhm, YX55069BCT2:R0402, symbol YX55069BCT2:RC0402FR-0710KL
- added R15, R16: 27 Ohm, YX55069BCT2:R0402, symbol YX55069BCT2:RC0402FR-0727RL
- added R17: 43.2 kOhm, YX55069BCT2:R0402, symbol YX55069BCT2:0402WGF4322TCE
- added R18, R19: 47k, YX55069BCT2:R_0603_1608Metric, symbol YX55069BCT2:R_100k_0603
- added R20: 100k, YX55069BCT2:R_0603_1608Metric, symbol YX55069BCT2:R_100k_0603
- added R21, R24: 1k, YX55069BCT2:R_0603_1608Metric, symbol YX55069BCT2:R_100k_0603
- added R23: 100 Ohm, YX55069BCT2:R0402, symbol YX55069BCT2:RC0402FR-07100RL
- added U13: SN74AXC1T45DCKR, slate113:SC-70-6_L2.0-W1.3-P0.65-LS2.1-BL-1, symbol slate113:SN74AXC1T45DCKR
- added U64: PCA9306DCUR, slate113:SSOP-8_L2.0-W2.3-P0.50-LS3.1-BR, symbol slate113:PCA9306DCUR
Connections:
- net 1V1 is gone; now on net 1V15: C26.2, C27.2, U7.1 (OUT)
- net VDD33_HDMI is gone; now on net 3V3: R1.2, U1.B1 (VDD33_HDMI)
- net 1V2: now also U1.B10 (VDD12_MIPI1), U1.J10 (VDD12_MIPI0), C39.2, C40.2, C49.2, C52.2
- net 1V8: now also R2.2, U1.J7 (VDDIO18), U4.2 (SNS), C16.2, C46.2, C50.2, R104.2, R106.1, U13.1 (VCCA), U13.5 (DIR), U64.2 (VREF1); no longer R2.1
- net 2V8: now also U5.2 (SNS)
- net D0+: now also D5.1 (IO1)
- net D0-: now also D5.2 (IO2)
- net D1+: now also D4.4 (IO3)
- net D1-: now also D4.5 (IO4)
- net D2+: now also D4.1 (IO1)
- net D2-: now also D4.2 (IO2)
- net DDC_SCL: now also D3.1 (D1+), R18.1
- net DDC_SDA: now also D3.2 (D1-), R19.1
- net ESP_DN: now also U12.6 (I/O1), R15.1; no longer U10.25 (GPIO19), U12.4 (I/O2)
- net ESP_DP: now also U12.4 (I/O2), R16.2; no longer U10.26 (GPIO20), U12.6 (I/O1)
- net GND: now also C2.1, C21.1, C24.1, U1.A10 (VSS), U1.C9 (VSS), U1.D4 (VSS), U1.D5 (VSS), U1.D6 (VSS), U1.D7 (VSS), U1.E4 (VSS), U1.E5 (VSS), U1.E6 (VSS), U1.E7 (VSS), U1.F4 (VSS), U1.F5 (VSS), U1.F6 (VSS), U1.F7 (VSS), U1.G4 (VSS), U1.G7 (VSS), U1.H1 (VSS), U1.K10 (VSS), C157.2, C16.1, C29.1, C30.2, C39.1, C40.1, C41.1, C42.1, C43.1, C44.1, C45.1, C46.1, C47.1, C48.1, C49.1, C50.1, C51.1, C52.1, C53.1, C54.1, C55.1, C56.1, C57.1, C58.1, C59.1, C60.1, C61.1, C62.1, D3.3 (GND), D3.8 (GND), D4.3 (GND), D4.8 (GND), D5.3 (GND), D5.8 (GND), Q2.2 (S), R107.1, R14.2, R20.2, U13.2 (GND), U64.1 (GND); no longer C10.1, C12.1, C150.1, C20.2, C21.2, C31.2, C33.2, C34.2, C35.2, C36.2, C4.2, C5.2, C6.2, FPC1.23, L3.1, R101.2, R6.1, R7.1, R99.2, U10.2 (VDD3P3), U10.20 (VDD3P3_RTC), U10.3 (VDD3P3), U10.46 (VDD3P3_CPU), U10.55 (VDDA), U10.56 (VDDA), U3.1 (VDD), U3.3 (CFG3), U6.1 (OUT), U63.3 (VIN), U9.22 (VDD), U9.7 (EN/VDDIO)
- net HDMICN: now also D5.5 (IO4)
- net HDMICP: now also D5.4 (IO3)
- net HDMI_5V_IN: now also D3.5 (D2-), R18.2, R19.2, R20.1
- net HPD0: now also R21.1; no longer J1.19 (HPD)
- net I2C0_SCL: now also R108.2, U64.6 (SCL2); no longer U1.K4 (I2C_SCL)
- net I2C0_SDA: now also U64.5 (SDA2); no longer U1.K3 (I2C_SDA)
- net LCD_PWM: now also U10.14 (GPIO9)
- net LCD_RST_L: now also Q2.3 (D)
- net VBUS: now also C30.1, R24.2; no longer U3.8 (VBUS)
- net VDD_SPI: now also C61.2
- net 3V3: now reaches U6.2 (SNS)
- net 3V3: now also C12.1, C150.1, C20.2, C21.2, C31.2, C33.2, C34.2, C35.2, C36.2, C4.2, C5.2, C6.2, FPC1.23, L3.1, R101.2, R6.1, R7.1, R99.2, U1.G1 (VDD33_HDMI), U1.H2 (VDDIO33), U10.2 (VDD3P3), U10.20 (VDD3P3_RTC), U10.3 (VDD3P3), U10.46 (VDD3P3_CPU), U10.55 (VDDA), U10.56 (VDDA), U6.1 (OUT), U63.3 (VIN), U9.22 (VDD), U9.7 (EN/VDDIO), C29.2, C43.2, C45.2, C48.2, C51.2, C57.2, C58.2, C59.2, C60.2, C62.2, R103.2, R108.1, U13.6 (VCCB); no longer C21.1
- net at OSC1.1 (Tri-state): now also R2.1; no longer R2.2
- net at C27.1, R5.2, U7.2 (FB): now also R17.1
- net HDMI_INT: now reaches U10.12 (GPIO7)
- net HDMI_INT: now also U13.4 (B)
- net LCD_RST_L_F: now reaches U10.13 (GPIO8)
- net LCD_RST_L_F: now also R23.2
- net 1V15: now reaches U1.B2 (VDD11_HDMI)
- net 1V15: now also U1.C10 (VDDC11), U1.G2 (VDD11_HDMI), U1.K6 (VDDC11), C41.2, C42.2, C44.2, C47.2, C53.2, C54.2, C55.2, C56.2, R17.2
- net INT: now reaches U1.J3 (INT)
- net INT: now also R14.1, U13.3 (A)
- net at U3.4 (DP): now also U3.5 (DM)
- new net: Q2.1 (G), R107.2, R23.1
- new net: C157.1, R103.1, U64.7 (VREF2), U64.8 (EN)
- new net: R16.1, U10.26 (GPIO20)
- new net: R15.2, U10.25 (GPIO19)
- new net: C10.1, R24.1, U3.1 (VDD)
- new net HDMI_SCL: R106.2, U1.K4 (I2C_SCL), U64.3 (SCL1)
- new net HDMI_SDA: R104.1, U1.K3 (I2C_SDA), U64.4 (SDA1)
- new net HPD: D3.4 (D2+), J1.19 (HPD), R21.2
- new net VDD: U3.3 (CFG3)
- no-connect marks 25 -> 76
Other:
- note added: "Decoupling"
- note added: "ESP32"
- note added: "HDMI -> MIPI BGA"
- note added: "USB-C"
- moved on the sheet: C14, C15, C31, C33, C35, C36, C37, C38, C4, C5, C8, C9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

Commit message: made final schematic changes
Parts:
- removed C11: 10µF, Capacitor_SMD:C_0603_1608Metric, symbol Device:C_Small
- removed C12: 2.2µF, Capacitor_SMD:C_0603_1608Metric, symbol Device:C_Small
- removed R10: 127kΩ, Resistor_SMD:R_0603_1608Metric, symbol Device:R
- removed R8: 205kΩ, Resistor_SMD:R_0603_1608Metric, symbol Device:R
- removed U9: LP8556SQ-E09/NOPB, slate113:WQFN-24_L4.0-W4.0-P0.50-BL-EP2.5, symbol slate113:LP8556SQ-E09_NOPB
- added C11: 1 nF, YX55069BCT2:C0402, symbol YX55069BCT2:CL05B102KB5NNNC
- added C12: 2.2 nF, YX55069BCT2:C0402, symbol YX55069BCT2:CL05B222KB5NNNC
- added C63, C64: 100nF, YX55069BCT2:C0603, symbol Device:C_Small
- added C65: 100 nF, YX55069BCT2:C_0603_1608Metric, symbol Device:C_Small
- added C66: 220 nF, YX55069BCT2:C0402, symbol YX55069BCT2:CL05B224KO5NNNC
- added C67: 4.7µF, YX55069BCT2:C0805, symbol Device:C_Small
- added C68: 1uF, YX55069BCT2:CL05A105KA5NQNC, symbol Device:C_Small
- added C69: 10uF, YX55069BCT2:C0603, symbol Device:C_Small
- added Q4: BSS138_C112239, YX55069BCT2:SOT-23-3_L2.9-W1.6-P1.90-LS2.8-BR, symbol YX55069BCT2:BSS138_C112239
- added R10: 31.6 kOhm, YX55069BCT2:R0402, symbol YX55069BCT2:0402WGF3162TCE
- added R110: 100kΩ, Resistor_SMD:R_0603_1608Metric, symbol Device:R_Small
- added R26: 1.10 kOhm, YX55069BCT2:R0402, symbol YX55069BCT2:0402WGF1101TCE
- added R27: 100 Ohm, YX55069BCT2:R0402, symbol YX55069BCT2:RC0402FR-07100RL
- added R28: 100 kOhm, YX55069BCT2:R0402, symbol YX55069BCT2:0402WGF1003TCE
- added R8: 348 kOhm, YX55069BCT2:R0402, symbol YX55069BCT2:0402WGF3483TCE
- added R9: 5 Ohm, YX55069BCT2:R0402, symbol YX55069BCT2:CSRT0402FT5R00
- added U14: TXS0101DBVR, YX55069BCT2:SOT-23-6_L2.9-W1.6-P0.95-LS2.8-BR, symbol YX55069BCT2:TXS0101DBVR
- added U15: TPS61165DBVR, YX55069BCT2:SOT-23-6_L2.9-W1.6-P0.95-LS2.8-BR, symbol YX55069BCT2:TPS61165DBVR
- added U16: TVS0500DRVR, YX55069BCT2:WSON-6_L2.0-W2.0-P0.65-BL-EP, symbol YX55069BCT2:TVS0500DRVR
- added U9: TPS259474LRPWR, YX55069BCT2:VQFN-10_L2.0-W2.0-P0.45-TL, symbol YX55069BCT2:TPS259474LRPWR
- C13: value 4.7µF -> 10 uF; footprint Capacitor_SMD:C_0603_1608Metric -> YX55069BCT2:C1206; LCSC Part C77045 -> C100122; MPN GRM188R61C475KE11D -> (none); Manufacturer Murata Electronics -> (none)
Connections:
- net 1V8: now also C63.2, U14.1 (VCCA), U14.5 (OE)
- net 3V3: now also C64.2, U14.6 (VCCB); no longer L3.1
- net GND: now also U3.3 (CFG3), C11.1, C12.2, C63.1, C64.1, C65.2, C66.1, C67.1, C68.1, C69.2, Q4.2 (S), R110.1, R26.1, R28.1, R9.2, U14.2 (GND), U15.4 (GND), U16.1 (GND), U16.2 (GND), U16.3 (GND), U16.7 (GND), U9.8 (GND); no longer U3.9 (CFG1)
- net L1P1: now also U15.3 (SW)
- net LCD_LED_K: now also R9.1, U15.6 (FB)
- net LCD_PWM: now also U15.2 (CTRL); no longer FPC1.18
- net TP_INT_L: now also U14.3 (A); no longer U10.7 (GPIO2)
- net TP_RST_L: now also Q4.3 (D); no longer U10.6 (GPIO1)
- net VBUS: now also C68.2, R8.2, U9.5 (IN); no longer C1.1, C19.1, C22.1, C25.1, C28.1, C30.1, U12.5 (VBUS), U2.4 (EN), U2.6 (IN), U4.4 (EN), U4.6 (IN), U5.4 (EN), U5.6 (IN), U6.4 (EN), U6.6 (IN), U7.4 (EN), U7.6 (IN)
- net VDD: now also C10.1, R24.1, U3.1 (VDD), U3.9 (CFG1); no longer U3.3 (CFG3)
- new net: Q4.1 (G), R110.2, R27.1
- new net: C66.2, U15.5 (COMP)
- new net: C11.2, U9.7 (DVDT)
- new net: R10.1, R8.1, U9.1 (EN/UVLO)
- new net: C12.1, U9.10 (ITIMER)
- new net: R10.2, R28.2, U9.2 (OVLO/OVCSEL)
- new net: R26.2, U9.9 (ILM)
- new net SYS_5V: C1.1, C19.1, C22.1, C25.1, C28.1, C30.1, C65.1, C67.2, C69.1, L3.1, U12.5 (VBUS), U15.1 (VIN), U16.4 (IN), U16.5 (IN), U16.6 (IN), U2.4 (EN), U2.6 (IN), U4.4 (EN), U4.6 (IN), U5.4 (EN), U5.6 (IN), U6.4 (EN), U6.6 (IN), U7.4 (EN), U7.6 (IN), U9.6 (OUT)
- new net TP_INT_L_F: U10.7 (GPIO2), U14.4 (B)
- new net TP_RST_L_F: R27.2, U10.6 (GPIO1)
- no-connect marks 76 -> 74
Other:
- note added: "Level Shifters"
- note added: "PD Controller"
- note added: "VBUS Protection"
- moved on the sheet: C10, Q2, R107, R23, R24, U3
