File: Kicad Project/_restore_backup_2026-09-30T10-44-40-514/YX55069BCT2-Driver-Board.kicad_sch (KiCad schematic)
At the start: 151 parts, among them J1 10029449-001RLF, Q1 BSS138_C112239, Q2 BSS138_C112239, Q4 BSS138_C112239, SW3 BOOT, SW4 RESET, U1 TC358870XBG(NOK), U10 ESP32-S3R8, U11 GD25Q128EWIGR, U12 USBLC6-2SC6, U13 SN74AXC1T45DCKR, U14 TXS0101DBVR, U15 TPS61165DBVR, U16 TVS0500DRVR, U2 TLV76701DRVR, U3 CH224K, U4 TLV76718DRVR, U5 TLV76728DRVR, U6 TLV76733DRVR, U62 PCA9306DCUR, U63 AP2120N-2.8TRG1, U64 PCA9306DCUR, U7 TLV76701DRVR, U8 ESD7104MUTAG_C2987068, U9 TPS259474LRPWR, X1 ABM8-40.000MHZ-10-D1G-T

Commit message: started PCB work + wire up most of the HDMI -> MIPI converter BGA & ESP32
Parts:
- FB1, FB2: footprint YX55069BCT2:L_0603_1608Metric -> YX55069BCT2:USB-C-SMD_TYPE-C16PIN
- R3, R4, R5: footprint Resistor_SMD:R_0805_2012Metric -> Resistor_THT:R_Array_SIP4
Connections:
- net FB1: no longer names the net of FB1.1, J1.SH
Other:
- moved on the sheet: C43, C45, C48, C51, C57, C58, C59, C60
